Commit message: hardware

File: mp_bot/mp_bot_description/urdf/robot.urdf.xacro (robot description, xacro)
@@ -1,4 +1,5 @@
 <?xml version="1.0"?>
 <robot xmlns:xacro="http://www.ros.org/wiki/xacro"  name="mp_bot">
+    <xacro:arg name="sim_mode" default="false"/>
     <xacro:include filename="mp_bot_links.xacro" />
     <xacro:include filename="mp_bot_joints.xacro" />

File: mp_bot/mp_bot_description/urdf/ros2_control.xacro (robot description, xacro)
@@ -10,25 +10,57 @@
     <param name="initial_value">-0.1</param>
   </xacro:macro>
-  <ros2_control name="GazeboSystem" type="system">
-    <hardware>
-        <plugin>gazebo_ros2_control/GazeboSystem</plugin>
-    </hardware>
-    <joint name="left_wheel_joint">
-        <command_interface name="velocity">
-            <param name="min">-10</param>
-            <param name="max">10</param>
-        </command_interface>
-        <state_interface name="velocity"/>
-        <state_interface name="position"/>
-    </joint>
-    <joint name="right_wheel_joint">
-        <command_interface name="velocity">
-            <param name="min">-10</param>
-            <param name="max">10</param>
-        </command_interface>
-        <state_interface name="velocity"/>
-        <state_interface name="position"/>
-    </joint>
-  </ros2_control>
+  <xacro:unless value="$(arg sim_mode)">
+      <ros2_control name="RealRobot" type="system">
+          <hardware>
+              <plugin>diffdrive_arduino/DiffDriveArduinoHardware</plugin>
+              <param name="left_wheel_name">left_wheel_joint</param>
+              <param name="right_wheel_name">right_wheel_joint</param>
+              <param name="loop_rate">30</param>
+              <param name="device">/dev/ttyACM0</param>
+              <param name="baud_rate">57600</param>
+              <param name="timeout_ms">1000</param>
+              <param name="enc_counts_per_rev">537.6</param>
+          </hardware>
+          <joint name="left_wheel_joint">
+              <command_interface name="velocity">
+                  <param name="min">-10</param>
+                  <param name="max">10</param>
+              </command_interface>
+              <state_interface name="position"/>
+              <state_interface name="velocity"/>
+          </joint>
+          <joint name="right_wheel_joint">
+              <command_interface name="velocity">
+                  <param name="min">-10</param>
+                  <param name="max">10</param>
+              </command_interface>
+              <state_interface name="position"/>
+              <state_interface name="velocity"/>
+          </joint>
+      </ros2_control>
+  </xacro:unless>
+  <xacro:if value="$(arg sim_mode)">
+    <ros2_control name="GazeboSystem" type="system">
+      <hardware>
+          <plugin>gazebo_ros2_control/GazeboSystem</plugin>
+      </hardware>
+      <joint name="left_wheel_joint">
+          <command_interface name="velocity">
+              <param name="min">-10</param>
+              <param name="max">10</param>
+          </command_interface>
+          <state_interface name="velocity"/>
+          <state_interface name="position"/>
+      </joint>
+      <joint name="right_wheel_joint">
+          <command_interface name="velocity">
+              <param name="min">-10</param>
+              <param name="max">10</param>
+          </command_interface>
+          <state_interface name="velocity"/>
+          <state_interface name="position"/>
+      </joint>
+    </ros2_control>
+  </xacro:if>
   <ros2_control name="fr_arm" type="system">
     <hardware>
